File: QS-09.kicad_sch (KiCad schematic)
At the start: 49 parts, among them J1 TYPE-C-31-M12_13, SW1 Rotary_Encoder_Switch_Chassis, SW10 MXSwitch, SW11 MXSwitch, SW12 SW_Push, SW2 MXSwitch, SW3 MXSwitch, SW4 MXSwitch, SW5 Rotary_Encoder_Switch_Chassis, SW6 MXSwitch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

Commit message: USB ready, fixed RGB
Connections:
- net GND: now also C4.2, C5.1
- net RGB: now also D16.4 (DIN), U1.25 (PC5); no longer D10.4 (DIN), U1.14 (PB0)
- net UNDERGLOW: now also D10.2 (DOUT), D21.4 (DIN); no longer D18.2 (DOUT), D19.4 (DIN)
- net at D22.2 (DOUT): now also D19.4 (DIN)
- net at D11.4 (DIN): now also D12.2 (DOUT); no longer D10.2 (DOUT)
- net at D15.2 (DOUT): now also D12.4 (DIN); no longer D16.4 (DIN)
- net at D15.4 (DIN): now also D18.2 (DOUT); no longer D14.2 (DOUT)
- net at D13.2 (DOUT): now also D10.4 (DIN); no longer D14.4 (DIN)
- net at D13.4 (DIN): now also D14.2 (DOUT); no longer D12.2 (DOUT)
- net at D20.2 (DOUT): no longer D21.4 (DIN)
- net at D11.2 (DOUT): now also D14.4 (DIN); no longer D12.4 (DIN)
Other:
- moved on the sheet: D10, D11, D12, D13, D14, D15, D16, D17, D18, D19, D20, D21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
Changed lines of the file:
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@@
   (junction (at 111.76 93.472) (diameter 1.016) (color 0 0 0 0))
   (junction (at 117.348 97.282) (diameter 1.016) (color 0 0 0 0))
+  (junction (at 117.348 98.552) (diameter 1.016) (color 0 0 0 0))
   (junction (at 117.602 170.688) (diameter 1.016) (color 0 0 0 0))
   (junction (at 117.602 185.928) (diameter 1.016) (color 0 0 0 0))
@@
     (stroke (width 0) (type solid) (color 0 0 0 0))
   )
-  (wire (pts (xy 111.76 98.552) (xy 122.428 98.552))
+  (wire (pts (xy 111.76 98.552) (xy 117.348 98.552))
     (stroke (width 0) (type solid) (color 0 0 0 0))
   )
@@
     (stroke (width 0) (type solid) (color 0 0 0 0))
   )
-  (wire (pts (xy 117.348 97.282) (xy 117.348 100.838))
+  (wire (pts (xy 117.348 97.282) (xy 117.348 98.552))
+    (stroke (width 0) (type solid) (color 0 0 0 0))
+  )
+  (wire (pts (xy 117.348 98.552) (xy 117.348 100.838))
+    (stroke (width 0) (type solid) (color 0 0 0 0))
+  )
+  (wire (pts (xy 117.348 98.552) (xy 122.428 98.552))
     (stroke (width 0) (type solid) (color 0 0 0 0))
   )
@@
     )
   )
-  (global_label "RGB" (shape input) (at 68.326 28.956 0) (fields_autoplaced)
+  (global_label "RGB" (shape input) (at 68.326 56.896 0) (fields_autoplaced)
     (effects (font (size 1.27 1.27)) (justify left))
-    (property "Intersheet References" "${INTERSHEET_REFS}" (id 0) (at 74.5491 28.8766 0)
+    (property "Intersheet References" "${INTERSHEET_REFS}" (id 0) (at 74.5491 56.8166 0)
       (effects (font (size 1.27 1.27)) (justify left) hide)
     )
@@
   (symbol (lib_id "LED:WS2812B") (at 117.602 178.308 0) (unit 1)
     (in_bom yes) (on_board yes)
-    (property "Reference" "D19" (id 0) (at 120.9041 172.0655 0)
+    (property "Reference" "D21" (id 0) (at 120.9041 172.0655 0)
       (effects (font (size 1.27 1.27)) (justify left))
     )
@@
   (symbol (lib_id "LED:WS2812B") (at 132.842 178.308 0) (unit 1)
     (in_bom yes) (on_board yes)
-    (property "Reference" "D20" (id 0) (at 136.1441 172.0655 0)
+    (property "Reference" "D22" (id 0) (at 136.1441 172.0655 0)
       (effects (font (size 1.27 1.27)) (justify left))
     )
@@
   (symbol (lib_id "acheronSymbols:SK6812MINI-E") (at 138.684 140.97 0) (unit 1)
     (in_bom yes) (on_board yes)
-    (property "Reference" "D10" (id 0) (at 143.0021 134.4735 0)
+    (property "Reference" "D16" (id 0) (at 143.0021 134.4735 0)
       (effects (font (size 1.27 1.27)) (justify left))
     )
@@
   (symbol (lib_id "LED:WS2812B") (at 148.082 178.308 0) (unit 1)
     (in_bom yes) (on_board yes)
-    (property "Reference" "D21" (id 0) (at 151.3841 172.0655 0)
+    (property "Reference" "D19" (id 0) (at 151.3841 172.0655 0)
       (effects (font (size 1.27 1.27)) (justify left))
     )
@@
   (symbol (lib_id "acheronSymbols:SK6812MINI-E") (at 153.924 140.97 0) (unit 1)
     (in_bom yes) (on_board yes)
-    (property "Reference" "D11" (id 0) (at 158.2421 134.4735 0)
+    (property "Reference" "D17" (id 0) (at 158.2421 134.4735 0)
       (effects (font (size 1.27 1.27)) (justify left))
     )
@@
   (symbol (lib_id "LED:WS2812B") (at 163.322 178.308 0) (unit 1)
     (in_bom yes) (on_board yes)
-    (property "Reference" "D22" (id 0) (at 166.6241 172.0655 0)
+    (property "Reference" "D20" (id 0) (at 166.6241 172.0655 0)
       (effects (font (size 1.27 1.27)) (justify left))
     )
@@
   (symbol (lib_id "acheronSymbols:SK6812MINI-E") (at 169.164 140.97 0) (unit 1)
     (in_bom yes) (on_board yes)
-    (property "Reference" "D12" (id 0) (at 173.4821 134.4735 0)
+    (property "Reference" "D18" (id 0) (at 173.4821 134.4735 0)
       (effects (font (size 1.27 1.27)) (justify left))
     )
@@
   (symbol (lib_id "acheronSymbols:SK6812MINI-E") (at 184.404 140.97 0) (unit 1)
     (in_bom yes) (on_board yes)
-    (property "Reference" "D13" (id 0) (at 188.7221 134.4735 0)
+    (property "Reference" "D15" (id 0) (at 188.7221 134.4735 0)
       (effects (font (size 1.27 1.27)) (justify left))
     )
@@
   (symbol (lib_id "acheronSymbols:SK6812MINI-E") (at 199.644 140.97 0) (unit 1)
     (in_bom yes) (on_board yes)
-    (property "Reference" "D14" (id 0) (at 203.9621 134.4735 0)
+    (property "Reference" "D12" (id 0) (at 203.9621 134.4735 0)
       (effects (font (size 1.27 1.27)) (justify left))
     )
@@
   (symbol (lib_id "acheronSymbols:SK6812MINI-E") (at 214.884 140.97 0) (unit 1)
     (in_bom yes) (on_board yes)
-    (property "Reference" "D15" (id 0) (at 219.2021 134.4735 0)
+    (property "Reference" "D11" (id 0) (at 219.2021 134.4735 0)
       (effects (font (size 1.27 1.27)) (justify left))
     )
@@
   (symbol (lib_id "acheronSymbols:SK6812MINI-E") (at 230.124 140.97 0) (unit 1)
     (in_bom yes) (on_board yes)
-    (property "Reference" "D16" (id 0) (at 234.4421 134.4735 0)
+    (property "Reference" "D14" (id 0) (at 234.4421 134.4735 0)
       (effects (font (size 1.27 1.27)) (justify left))
     )
@@
   (symbol (lib_id "acheronSymbols:SK6812MINI-E") (at 245.364 140.97 0) (unit 1)
     (in_bom yes) (on_board yes)
-    (property "Reference" "D17" (id 0) (at 249.6821 134.4735 0)
+    (property "Reference" "D13" (id 0) (at 249.6821 134.4735 0)
       (effects (font (size 1.27 1.27)) (justify left))
     )
@@
   (symbol (lib_id "acheronSymbols:SK6812MINI-E") (at 260.604 140.97 0) (unit 1)
     (in_bom yes) (on_board yes)
-    (property "Reference" "D18" (id 0) (at 264.9221 134.4735 0)
-      (effects (font (size 1.27 1.27)) (justify left))
-    )
+    (property "Reference" "D10" (id 0) (at 264.9221 134.4735 0)
+      (effects (font (size 1.27 1.27)) (justify left))
+    )

Commit message: alpha
Parts:
- removed R3: 10k, Resistor_SMD:R_0603_1608Metric, symbol Device:R_Small
- removed SW12: SW_Push, Button_Switch_SMD:SW_SPST_SKQG_WithStem, symbol Switch:SW_Push
- SW1, SW5: value Rotary_Encoder_Switch_Chassis -> Encoder
Connections:
- net COL0: now also U1.23 (PC6)
- net COL1: now also U1.13 (~HWB~/PD7)
- net COL2: now also U1.19 (PB5)
- net GND: now also SW1.C, SW5.C
- net ROW0: now also U1.7 (PD1)
- net ROW1: now also U1.8 (PD2)
- net ROW2: now also U1.20 (PB6)
- net ENCA1: now reaches SW1.A
- net ENCA1: now also U1.21 (PB7)
- net ENCB1: now reaches SW1.B
- net ENCB1: now also U1.22 (PC7)
- net ENCB2: now reaches U1.10 (PD4)
- net ENCB2: now also SW5.B
- net ENCA2: now reaches U1.9 (PD3)
- net ENCA2: now also SW5.A
- no-connect marks 3 -> 15
Other:
- moved on the sheet: SW1, SW5

Commit message: Added reset button, fixed a missing resistor
Parts:
- added R3, R6: 10k, Resistor_SMD:R_0603_1608Metric, symbol Device:R_Small
- added SW12: SW_Push, Button_Switch_SMD:SW_SPST_SKQG_WithStem, symbol Switch:SW_Push
Connections:
- net +5V: now also R6.1
- net COL1: now also U1.14 (PB0); no longer U1.13 (~HWB~/PD7)
- net GND: now also R3.2, SW12.1
- net RESET: now also R6.2, SW12.2
- new net: R3.1, U1.13 (~HWB~/PD7)
- no-connect marks 15 -> 14
Changed lines of the file:
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@@
   (junction (at 92.964 88.9) (diameter 1.016) (color 0 0 0 0))
   (junction (at 92.964 95.504) (diameter 1.016) (color 0 0 0 0))
+  (junction (at 109.728 120.142) (diameter 1.016) (color 0 0 0 0))
   (junction (at 111.76 93.472) (diameter 1.016) (color 0 0 0 0))
   (junction (at 117.348 97.282) (diameter 1.016) (color 0 0 0 0))
@@
   (no_connect (at 56.642 170.942))
   (no_connect (at 56.642 173.482))
-  (no_connect (at 68.326 28.956))
   (no_connect (at 68.326 31.496))
   (no_connect (at 68.326 34.036))
@@
     (stroke (width 0) (type solid) (color 0 0 0 0))
   )
+  (wire (pts (xy 68.326 89.916) (xy 68.326 91.948))
+    (stroke (width 0) (type solid) (color 0 0 0 0))
+  )
+  (wire (pts (xy 68.326 91.948) (xy 73.406 91.948))
+    (stroke (width 0) (type solid) (color 0 0 0 0))
+  )
   (wire (pts (xy 85.852 88.9) (xy 85.852 90.424))
     (stroke (width 0) (type solid) (color 0 0 0 0))
@@
   )
   (wire (pts (xy 100.076 88.9) (xy 100.076 90.424))
+    (stroke (width 0) (type solid) (color 0 0 0 0))
+  )
+  (wire (pts (xy 104.14 120.142) (xy 109.728 120.142))
+    (stroke (width 0) (type solid) (color 0 0 0 0))
+  )
+  (wire (pts (xy 109.728 116.586) (xy 109.728 120.142))
+    (stroke (width 0) (type solid) (color 0 0 0 0))
+  )
+  (wire (pts (xy 109.728 120.142) (xy 112.268 120.142))
     (stroke (width 0) (type solid) (color 0 0 0 0))
   )
@@
     )
   )
+  (global_label "COL1" (shape input) (at 68.326 28.956 0) (fields_autoplaced)
+    (effects (font (size 1.27 1.27)) (justify left))
+    (property "Intersheet References" "${INTERSHEET_REFS}" (id 0) (at 75.5772 28.8766 0)
+      (effects (font (size 1.27 1.27)) (justify left) hide)
+    )
+  )
   (global_label "COL2" (shape input) (at 68.326 41.656 0) (fields_autoplaced)
     (effects (font (size 1.27 1.27)) (justify left))
@@
     (effects (font (size 1.27 1.27)) (justify left))
     (property "Intersheet References" "${INTERSHEET_REFS}" (id 0) (at 76.9681 77.2954 0)
-      (effects (font (size 1.27 1.27)) (justify left) hide)
-    )
-  )
-  (global_label "COL1" (shape input) (at 68.326 84.836 0) (fields_autoplaced)
-    (effects (font (size 1.27 1.27)) (justify left))
-    (property "Intersheet References" "${INTERSHEET_REFS}" (id 0) (at 75.5772 84.7566 0)
       (effects (font (size 1.27 1.27)) (justify left) hide)
     )
@@
     )
   )
+  (global_label "RESET" (shape input) (at 112.268 120.142 0) (fields_autoplaced)
+    (effects (font (size 1.27 1.27)) (justify left))
+    (property "Intersheet References" "${INTERSHEET_REFS}" (id 0) (at 120.4263 120.0626 0)
+      (effects (font (size 1.27 1.27)) (justify left) hide)
+    )
+  )
   (global_label "COL2" (shape input) (at 121.412 33.782 90) (fields_autoplaced)
     (effects (font (size 1.27 1.27)) (justify left))
@@
     (pin "1")
   )
+  (symbol (lib_id "power:+5V") (at 109.728 111.506 0) (unit 1)
+    (in_bom yes) (on_board yes) (fields_autoplaced)
+    (property "Reference" "#PWR010" (id 0) (at 109.728 115.316 0)
+      (effects (font (size 1.27 1.27)) hide)
+    )
+    (property "Value" "+5V" (id 1) (at 109.728 107.9014 0))
+    (property "Footprint" "" (id 2) (at 109.728 111.506 0)
+      (effects (font (size 1.27 1.27)) hide)
+    )
+    (property "Datasheet" "" (id 3) (at 109.728 111.506 0)
+      (effects (font (size 1.27 1.27)) hide)
+    )
+    (pin "1")
+  )
   (symbol (lib_id "power:+5V") (at 112.522 170.688 90) (unit 1)
     (in_bom yes) (on_board yes) (fields_autoplaced)
@@
     (pin "1")
   )
+  (symbol (lib_id "power:GND") (at 73.406 91.948 0) (unit 1)
+    (in_bom yes) (on_board yes) (fields_autoplaced)
+    (property "Reference" "#PWR08" (id 0) (at 73.406 98.298 0)
+      (effects (font (size 1.27 1.27)) hide)
+    )
+    (property "Value" "GND" (id 1) (at 73.406 96.5106 0))
+    (property "Footprint" "" (id 2) (at 73.406 91.948 0)
+      (effects (font (size 1.27 1.27)) hide)
+    )
+    (property "Datasheet" "" (id 3) (at 73.406 91.948 0)
+      (effects (font (size 1.27 1.27)) hide)
+    )
+    (pin "1")
+  )
   (symbol (lib_id "power:GND") (at 90.17 162.814 0) (unit 1)
     (in_bom yes) (on_board yes) (fields_autoplaced)
@@
     )
     (property "Datasheet" "" (id 3) (at 92.964 95.504 0)
+      (effects (font (size 1.27 1.27)) hide)
+    )
+    (pin "1")
+  )
+  (symbol (lib_id "power:GND") (at 93.98 120.142 0) (unit 1)
+    (in_bom yes) (on_board yes) (fields_autoplaced)
+    (property "Reference" "#PWR019" (id 0) (at 93.98 126.492 0)
+      (effects (font (size 1.27 1.27)) hide)
+    )
+    (property "Value" "GND" (id 1) (at 93.98 124.7046 0))
+    (property "Footprint" "" (id 2) (at 93.98 120.142 0)
+      (effects (font (size 1.27 1.27)) hide)
+    )
+    (property "Datasheet" "" (id 3) (at 93.98 120.142 0)
       (effects (font (size 1.27 1.27)) hide)
     )
@@
     (pin "2")
   )
+  (symbol (lib_id "Device:R_Small") (at 68.326 87.376 0) (unit 1)
+    (in_bom yes) (on_board yes) (fields_autoplaced)
+    (property "Reference" "R3" (id 0) (at 69.8247 86.4675 0)
+      (effects (font (size 1.27 1.27)) (justify left))
+    )
+    (property "Value" "10k" (id 1) (at 69.8247 89.2426 0)
+      (effects (font (size 1.27 1.27)) (justify left))
+    )
+    (property "Footprint" "Resistor_SMD:R_0603_1608Metric" (id 2) (at 68.326 87.376 0)
+      (effects (font (size 1.27 1.27)) hide)
+    )
+    (property "Datasheet" "~" (id 3) (at 68.326 87.376 0)
+      (effects (font (size 1.27 1.27)) hide)
+    )
+    (pin "1")
+    (pin "2")
+  )
+  (symbol (lib_id "Device:R_Small") (at 109.728 114.046 0) (unit 1)
+    (in_bom yes) (on_board yes) (fields_autoplaced)
+    (property "Reference" "R6" (id 0) (at 111.2267 113.1375 0)
+      (effects (font (size 1.27 1.27)) (justify left))
+    )
+    (property "Value" "10k" (id 1) (at 111.2267 115.9126 0)
+      (effects (font (size 1.27 1.27)) (justify left))
+    )
+    (property "Footprint" "Resistor_SMD:R_0603_1608Metric" (id 2) (at 109.728 114.046 0)
+      (effects (font (size 1.27 1.27)) hide)
+    )
+    (property "Datasheet" "~" (id 3) (at 109.728 114.046 0)
+      (effects (font (size 1.27 1.27)) hide)
+    )
+    (pin "1")
+    (pin "2")
+  )
   (symbol (lib_id "Device:D_Small") (at 166.878 37.846 270) (unit 1)
     (in_bom yes) (on_board yes) (fields_autoplaced)
@@
     (pin "3")
     (pin "4")
+  )
+  (symbol (lib_id "Switch:SW_Push") (at 99.06 120.142 0) (unit 1)
+    (in_bom yes) (on_board yes) (fields_autoplaced)
+    (property "Reference" "SW12" (id 0) (at 99.06 113.2544 0))
+    (property "Value" "SW_Push" (id 1) (at 99.06 116.0295 0))
+    (property "Footprint" "Button_Switch_SMD:SW_SPST_SKQG_WithStem" (id 2) (at 99.06 115.062 0)
+      (effects (font (size 1.27 1.27)) hide)
+    )
+    (property "Datasheet" "~" (id 3) (at 99.06 115.062 0)
+      (effects (font (size 1.27 1.27)) hide)
+    )
+    (pin "1")
+    (pin "2")
   )
   (symbol (lib_id "acheronSymbols:Rotary_Encoder_Switch_Chassis") (at 98.298 41.656 90) (unit 1)
@@
       (reference "#PWR07") (unit 1) (value "+5V") (footprint "")
     )
+    (path "/1ac041d6-778a-4241-a8d2-1db6617aff37"
+      (reference "#PWR08") (unit 1) (value "GND") (footprint "")
+    )
     (path "/2b0ec766-ec27-4459-a952-b19088911cb3"
       (reference "#PWR09") (unit 1) (value "GND") (footprint "")
     )
+    (path "/f7fc52f1-6355-4783-88b7-a094ce9a6b45"
+      (reference "#PWR010") (unit 1) (value "+5V") (footprint "")
+    )
     (path "/54af1ea5-6b9a-4268-bd58-88bda8abeaf0"
       (reference "#PWR011") (unit 1) (value "GND") (footprint "")
@@
       (reference "#PWR018") (unit 1) (value "GND") (footprint "")
     )
+    (path "/fd007b87-7236-412a-9d9e-e91195a95e5b"
+      (reference "#PWR019") (unit 1) (value "GND") (footprint "")
+    )
     (path "/3de74ab2-0ebc-4c88-9606-aaa555b4b2bd"
       (reference "#PWR0101") (unit 1) (value "GND") (footprint "")
@@
       (reference "R2") (unit 1) (value "22") (footprint "Resistor_SMD:R_0603_1608Metric")
     )
+    (path "/a6d1210a-53fd-4d11-9a29-99698184cf64"
+      (reference "R3") (unit 1) (value "10k") (footprint "Resistor_SMD:R_0603_1608Metric")
+    )
     (path "/27331b0e-0495-46c8-9952-41302f0163d2"
       (reference "R4") (unit 1) (value "5.1k") (footprint "Resistor_SMD:R_0603_1608Metric")
@@
       (reference "R5") (unit 1) (value "5.1k") (footprint "Resistor_SMD:R_0603_1608Metric")
     )
+    (path "/b98c031a-8b43-4b2e-845d-8e0c9bd9eca6"
+      (reference "R6") (unit 1) (value "10k") (footprint "Resistor_SMD:R_0603_1608Metric")
+    )
     (path "/874cedd9-1f2d-41e1-94c1-530f0b172b5c"
       (reference "SW1") (unit 1) (value "Encoder") (footprint "Rotary_Encoder:RotaryEncoder_Alps_EC11E-Switch_Vertical_H20mm")
@@
       (reference "SW11") (unit 1) (value "MXSwitch") (footprint "acheron_MX_SolderMask:MX100")
     )
+    (path "/97b38bd3-a371-4247-b664-f635af31146a"
+      (reference "SW12") (unit 1) (value "SW_Push") (footprint "Button_Switch_SMD:SW_SPST_SKQG_WithStem")
+    )
     (path "/a363adff-866e-49c2-903f-1e373fbbebf8"

Commit message: Fixed some wonky shit with the data lines
Connections:
- net UD+: now also J1.A6 (D+), J1.B6 (D+); no longer J1.A7 (D-), J1.B7 (D-)
- net UD-: now also J1.A7 (D-), J1.B7 (D-); no longer J1.A6 (D+), J1.B6 (D+)
Changed lines of the file:
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@@
     )
   )
-  (global_label "UD+" (shape input) (at 58.166 145.542 0) (fields_autoplaced)
+  (global_label "UD-" (shape input) (at 58.166 145.542 0) (fields_autoplaced)
     (effects (font (size 1.27 1.27)) (justify left))
     (property "Intersheet References" "${INTERSHEET_REFS}" (id 0) (at 64.752 145.4626 0)
@@
     )
   )
-  (global_label "UD-" (shape input) (at 58.166 153.162 0) (fields_autoplaced)
+  (global_label "UD+" (shape input) (at 58.166 153.162 0) (fields_autoplaced)
     (effects (font (size 1.27 1.27)) (justify left))
     (property "Intersheet References" "${INTERSHEET_REFS}" (id 0) (at 64.752 153.0826 0)
